File: auxiliary_converter.kicad_sch (KiCad schematic)
At the start: 0 parts

Commit message: Added auxiliary converter
Parts:
- added C45, C46, C49, C7: 1000uF/10V, symbol Device:C_Polarized
- added C48, C50, C57: 10uF/50V, symbol Device:C_Polarized
- added C51, C54, C56: 100nF, symbol Device:C
- added C52: 47nF, symbol Device:C
- added C53: 2.2nF, symbol Device:C
- added C57: 1nF, symbol Device:C
- added C58: 10nF, symbol Device:C
- added D14: PKC-136, symbol lib:PKC-136
- added D15: 1N5822, Diode_THT:D_DO-201AD_P15.24mm_Horizontal, symbol Diode:1N5822
- added D16: 1N5821, Diode_THT:D_DO-201AD_P15.24mm_Horizontal, symbol Diode:1N5821
- added D17: LL4148, Diode_SMD:D_MiniMELF, symbol Diode:LL4148
- added D18: BZV55B10, Diode_SMD:D_MiniMELF, symbol Diode:BZV55B10
- added D19: BZV55C30, Diode_SMD:D_MiniMELF, symbol Diode:BZV55C30
- added D20: BAV103, symbol lib:BAV103
- added D21, D23: B-15V, Diode_SMD:D_MiniMELF, symbol Diode:BZV55B15
- added D22: C-15V, Diode_SMD:D_MiniMELF, symbol Diode:BZV55C15
- added D?: BZV55C12, Diode_SMD:D_MiniMELF, symbol Diode:BZV55C12
- added J3: CON10, symbol lib:CON10
- added L7, L8: 33uH, symbol Device:L_Iron
- added Q10, Q8: BC847C, Package_TO_SOT_SMD:SOT-23, symbol Transistor_BJT:BC847
- added Q11: BC557C, Package_TO_SOT_THT:TO-92_Inline, symbol Transistor_BJT:BC557
- added Q7: BC547C, Package_TO_SOT_THT:TO-92_Inline, symbol Transistor_BJT:BC547
- added Q9: BC857C, symbol lib:BC857C
- added R62: 47, symbol Device:R
- added R64: 1.6k, symbol Device:R
- added R66, R67: 1k, symbol Device:R
- added R68: 22k, symbol Device:R
- added R69: 0R, symbol Device:R
- added R70: 22R, symbol Device:R
- added R71, R72, R74: 10k, symbol Device:R
- added R73: 8.2k, symbol Device:R
- added R75, R76, R84: 150k, symbol Device:R
- added R77: 4.7k, symbol Device:R
- added R79: 2.2k, symbol Device:R
- added R80, R81: 30k, symbol Device:R
- added R82: 100k, symbol Device:R
- added R83: 1M, symbol Device:R
- added U5: VIPER-12A, symbol lib:VIPER-12A
- added U6, U8: SFH617A-2, Package_DIP:DIP-4_W7.62mm, symbol Isolator:SFH617A-2
- added U7: TL431, Package_SO:SOIC-8_3.9x4.9mm_P1.27mm, symbol Reference_Voltage:TL431D
Connections:
- new net: C58.1, Q11.2 (B), R83.1, R84.1
- new net: R62.2, R67.1, U6.1
- new net: C45.1, D15.1 (K), L7.1
- new net: C7.1, D16.1 (K), L8.1
- new net: C49.1, C51.1, J3.7, J3.8, L8.2, R64.1
- new net: C52.1, D18.2 (A), D19.2 (A), U5.3 (FB)
- new net: C48.1, D17.1 (K), Q11.3 (E), U5.4 (VDD)
- new net: D14.2 (A), U5.5 (DRAIN), U5.6 (DRAIN), U5.7 (DRAIN), U5.8 (DRAIN)
- new net: C51.2, C53.2, C54.2, R64.2, R77.1, U7.8 (REF)
- new net: C57.1, D22.1 (K), Q7.2 (B), R74.1, U8.4
- new net: Q7.3 (E), R70.2
- new net: D14.1 (K), D?.1 (K)
- new net: C54.1, R73.2
- new net: D21.1 (K), D23.1 (K), Q8.2 (E), R75.1, R80.1, R81.1, R82.1
- new net: C56.1, D21.2 (A), D23.2 (A), Q10.1 (B), Q9.3 (C), R79.1
- new net: Q10.3 (C), Q9.1 (B), R72.2
- new net: Q9.2 (E), R69.1, R72.1, U8.2
- new net: R66.1, U8.1
- new net: C53.1, R67.2, R73.1, U6.2, U7.1 (K)
- new net: Q8.3 (C), R69.2
- new net: D17.2 (A), D18.1 (K), U6.3
- new net: R75.2, R76.1
- new net: Q8.1 (B), R71.1
- new net +200: R76.2
- new net +5Vst-by: C46.1, J3.1, J3.2, L7.2, R62.1, R66.2, R68.1
- new net +75: R82.2
- new net 0: C45.2, C46.2, C49.2, C56.2, C7.2, J3.10, J3.3, J3.4, J3.5, J3.6, Q10.2 (E), R77.2, R79.2, R80.2, R81.2, U7.2 (A), U7.3 (A), U7.6 (A), U7.7 (A)
- new net Earth: C48.2, C50.2, C52.2, C57.2, C57.2, C58.2, D22.2 (A), Q11.1 (C), R84.2, U5.1 (SOURCE), U5.2 (SOURCE), U8.3
- new net St-By: J3.9, R68.2, R71.2
- new net Vaux: C57.1, R70.1
- new net Vdc: D?.2 (A), R83.2
- new net Vs: C50.1, D19.1 (K), D20.1 (K), Q7.1 (C), R74.2, U6.4
Other:
- note added: "+3V3"
- note added: "+5Vst-by"
