File: resonant_converter.kicad_sch (KiCad schematic)
At the start: 0 parts

Commit message: Added resonant converter
Parts:
- added C23, C27, C32: 100n, symbol Device:C
- added C24, C60, C61: 470n, symbol Device:C
- added C25: 22u, symbol Device:C
- added C26: 270p, symbol Device:C
- added C28, C44, C59: 47n, symbol Device:C
- added C29, C30: 100u, symbol Device:C
- added C31, C41: 10u, symbol Device:C
- added C33: 4.7n, symbol Device:C
- added C34: 220p, symbol Device:C
- added C35: 47u, symbol Device:C
- added C37, C38: 220u, symbol Device:C
- added C39: 1u, symbol Device:C
- added C40: 10n, symbol Device:C
- added D10A, D10B: STTH1002C, symbol Device:D_Schottky_Dual_CommonAnode_KKA_Parallel
- added D11, D12, D7, D9: LL4148, Diode_SMD:D_MiniMELF, symbol Diode:LL4148
- added D13: C-12V, Diode_SMD:D_MiniMELF, symbol Diode:BZV55B12
- added D8A, D8B: BYT08P-400, symbol Device:D
- added J2: ~, symbol lib:CON8
- added L5: 10u, symbol Device:L_Iron
- added L6: 22u, symbol Device:L_Iron
- added Q4: BC557, Package_TO_SOT_THT:TO-92_Inline, symbol Transistor_BJT:BC557
- added Q5: NMOS, symbol Simulation_SPICE:NMOS
- added Q6: STP14NK50Z, symbol Simulation_SPICE:NMOS
- added R12: R, symbol Device:R
- added R33, R36, R39: 0, symbol Device:R
- added R34, R61: 2.7k, symbol Device:R
- added R35, R38, R40: 47, symbol Device:R
- added R37: 2.2Meg, symbol Device:R
- added R41: 16k, symbol Device:R
- added R42: 10, symbol Device:R
- added R43: 150, symbol Device:R
- added R46: 1.5k, symbol Device:R
- added R47: 10k, symbol Device:R
- added R48, R49, R50: 56k, symbol Device:R
- added R52: 3.3k, symbol Device:R
- added R53, R58: 75k, symbol Device:R
- added R56, R59: 1k, symbol Device:R
- added R60: 6.2k, symbol Device:R
- added R86: 470, symbol Device:R
- added R87: 220, symbol Device:R
- added R88: 560k, symbol Device:R
- added T1: T-RES-ER49-400W, symbol lib:T-RES-ER49-400W
- added U2: L6599, symbol Regulator_Controller:L6599
- added U3: SFH617A-2, Package_DIP:DIP-4_W7.62mm, symbol Isolator:SFH617A-2
- added U4: TL431D, Package_SO:SOIC-8_3.9x4.9mm_P1.27mm, symbol Reference_Voltage:TL431D
Connections:
- new net: C29.1, C30.1, C59.1, D8A.1 (K), D8B.1 (K), L5.1, R53.1
- new net: C30.2, C37.1, C38.1, D10A.1 (K), D10A.2 (K), D10B.1 (K), D10B.2 (K), L6.1, R48.1, R49.1, R50.1, T1.4 (SB), T1.5 (SC)
- new net: D10A.3 (A), T1.7 (SE)
- new net: C60.2, R87.1
- new net: C28.1, C34.1, T1.2 (AB)
- new net: C34.2, R43.1
- new net: C61.2, Q4.2 (B), R88.1
- new net: R52.2, R56.1, U3.1
- new net: C44.1, R56.2, U3.2, U4.1 (K)
- new net: C60.1, R46.2, U3.4
- new net: C44.2, R59.1
- new net: R58.2, R59.2, R60.1, R61.1, R86.2, U4.8 (REF)
- new net: D7.1 (K), R35.1, U2.15 (HVG)
- new net: Q5.2 (G), R33.2, R35.2
- new net: C23.2, Q4.3 (E), R34.1, R36.1, R88.2
- new net: C27.2, Q5.3 (S), Q6.1 (D), T1.1 (AA), U2.14 (OUT)
- new net: Q6.2 (G), R39.1, R40.1
- new net: D9.1 (K), R40.2, U2.11 (LVG)
- new net: D9.2 (A), R39.2
- new net: C41.1, D13.1 (K), R48.2, R49.2, R50.2, R52.1
- new net: D11.1 (K), D12.2 (A), R43.2
- new net: R53.2, R58.1
- new net: C33.1, R42.2, U2.7 (LINE)
- new net: C31.1, C32.1, R38.2, U2.12 (VCC)
- new net: D8B.2 (A), T1.6 (SD)
- new net: C39.1, D12.1 (K), R12.1, U2.6 (ISEN)
- new net: D7.2 (A), R33.1
- new net: R34.2, R41.2, R46.1, U2.4 (RFMIN), U2.5 (STBY)
- new net: D8A.2 (A), T1.3 (SA)
- new net: R36.2, U2.1 (CSS)
- new net: C27.1, U2.16 (VBOOT)
- new net: C24.2, R37.2, U2.2 (DELAY)
- new net: C26.2, U2.3 (CF)
- new net: C59.2, R86.1
- new net: D10B.3 (A), T1.10 (SH)
- new net +200V: C25.1, J2.1, J2.2, L5.2
- new net +75V: C35.1, J2.7, J2.8, L6.2
- new net Earth: C23.1, C24.1, C26.1, C28.2, C31.2, C32.2, C33.2, C39.2, C40.2, C61.1, D11.2 (A), Q4.1 (C), Q6.3 (S), R12.2, R37.1, R41.1, R47.2, R87.2, U2.10 (GND), U3.3
- new net GND: C25.2, C29.2, C35.2, C37.2, C38.2, C41.2, D13.2 (A), J2.3, J2.4, J2.5, J2.6, R60.2, R61.2, T1.8 (SF), T1.9 (SG), U4.2 (A), U4.3 (A), U4.6 (A), U4.7 (A)
- new net LINE: R42.1
- new net PWM-Latch: C40.1, R47.1, U2.8 (DIS)
- new net Vaux: R38.1
- new net Vdc: Q5.1 (D)
- no-connect marks 0 -> 1
